Commit message: arduino codes

File: src/main_delta_urdf/urdf/ros2_control_config.xacro (robot description, xacro)
@@ -8,5 +8,5 @@
      <!-- <plugin>delta_stepper_hw/DeltaStepperHardware</plugin> -->
     </hardware>
-    <joint name="link_0_JOINT_1">
+    <!-- <joint name="link_0_JOINT_1">
       <command_interface name="position"/>
       <state_interface name="position"/>
@@ -22,4 +22,28 @@
       <state_interface name="position"/>
       <state_interface name="velocity"/>
+    </joint> -->
+    <joint name="link_0_JOINT_1">
+      <command_interface name="position"/>
+      <command_interface name="velocity"/>    <!-- ← ADD THIS -->
+      <state_interface name="position">
+        <param name="initial_value">0.0</param>
+      </state_interface>
+      <state_interface name="velocity"/>
+    </joint>
+    <joint name="link_0_JOINT_2">
+      <command_interface name="position"/>
+      <command_interface name="velocity"/>    <!-- ← ADD THIS -->
+      <state_interface name="position">
+        <param name="initial_value">0.0</param>
+      </state_interface>
+      <state_interface name="velocity"/>
+    </joint>
+    <joint name="link_0_JOINT_3">
+      <command_interface name="position"/>
+      <command_interface name="velocity"/>    <!-- ← ADD THIS -->
+      <state_interface name="position">
+        <param name="initial_value">0.0</param>
+      </state_interface>
+      <state_interface name="velocity"/>
     </joint>
   </ros2_control>
